Commit message: iiwa14: Drake-family inertial swap (byte-identical grid.cuh vs GATO; regen via GATO vendored generator; gates 4/4 in-band)

File: tools/iiwa14.urdf (robot description, URDF)
Before this commit: robot KUKAiiwa14, 10 links, 9 joints
Links:
- link L1: mass 3.94781 -> 5.76
- link L2: mass 4.50275 -> 6.35
- link L3: mass 2.45520 -> 3.5
- link L4: mass 2.61155 -> 3.5
- link L5: mass 3.41000 -> 3.5
- link L6: mass 3.38795 -> 1.8
- link L7: mass 0.35432 -> 1.2
- link contact: mass 0.057 -> 0
